File: MultiSpork/hardware/MultiSpork-board/MultiSpork-v1.brd (EAGLE design)
At the start: 86.4 x 76.2 mm, 216 parts, among them J1 U.FL, Q2 32.768 kHz, Q3 40 MHz, Q4 MMBT3904, Q5 MMBT3904, SW1 JS102011SAQN, U1 USD-SOCKETNEW, U10 M25PX80, U2 SAM3SA-MU, U3 MAX11300GTL, U4 LT3580EMS8E, U5 LT3580EMS8E, U6 LT3580EMS8E, U7 MCP73831, U8 LT3580EMS8E, U9 CC3100

Commit message: Finished routing
Parts:
- moved R40 70.6 mm to (75.9, 63.5)
- moved C21 3.56 mm to (60.5, 40.1)
- moved C27 2.03 mm to (60.5, 36.8)
- moved C15 1.08 mm to (57.4, 46.2)
- moved C78 0.92 mm to (54.6, 18.5)
- moved ERASE 0.76 mm to (50.3, 52.6)
- moved JTAGSEL 0.76 mm to (53.1, 52.6)
- moved C79 0.72 mm to (54.6, 12.4)
- moved C73 0.51 mm to (41.7, 17.3)
- moved R31 0.51 mm to (41.7, 19.1)
- moved C80 0.32 mm to (52.3, 9.40)
- moved C29 0.25 mm to (60.5, 45.7)
- moved C32 0.25 mm to (64.0, 45.7)
- moved C30 0.06 mm to (60.5, 43.8)
Connections:
- net N$115 renamed D1P
- net N$116 renamed D1N
- net N$117 renamed D0N
- net N$118 renamed D0P
- net N$19 renamed PLL-GND
- net N$32 renamed ADC_REF
- net N$33 renamed DAC_REF
- net N$34 renamed PORT00'
- net N$35 renamed PORT01'
- net N$36 renamed PORT02'
- net N$37 renamed PORT03'
- net N$38 renamed PORT04'
- net N$39 renamed PORT05'
- net N$40 renamed PORT06'
- net N$41 renamed PORT07'
- net N$42 renamed PORT08'
- net N$43 renamed PORT09'
- net N$44 renamed PORT10'
- net N$45 renamed PORT11'
- net N$46 renamed PORT12'
- net N$47 renamed PORT13'
- net N$49 renamed PORT14'
- net N$50 renamed PORT15'
- net N$51 renamed PORT16'
- net N$52 renamed PORT17'
- net N$53 renamed PORT18'
- net N$54 renamed PORT19'
- net N$56 renamed VDD_IO
- net N$79 renamed VIN_IO2
- net N$80 renamed VIN_DIG
- net N$81 renamed VIN_ANA
- net N$83 renamed VIN_PA
- net N$84 renamed ANA_SW
- net N$85 renamed VDD_PA
- net N$87 renamed PA_SWP
- net N$88 renamed PA_SWN
- net N$90 renamed VDD_DIG
- net N$92 renamed VDD_RAM
- net N$93 renamed VDD_PLL
Routing:
- net +5V: track 4.24 -> 143.4 mm, vias 0 -> 8
- net V+: track 0.00 -> 119.7 mm, vias 0 -> 6
- net SHTDWN: track 0.00 -> 86.5 mm, vias 0 -> 6
- net VDD_IO: track 10.4 -> 82.4 mm, vias 1 -> 6
- net N$99: track 0.00 -> 66.2 mm, vias 0 -> 1
- net CC_INT: track 2.42 -> 58.7 mm, vias 0 -> 4
- net CC_RST: track 0.00 -> 55.4 mm, vias 0 -> 3
- net +3V3: track 57.1 -> 112.2 mm, vias 10 -> 28
- net N$109: track 0.00 -> 54.2 mm, vias 0 -> 1
- net CC_CS: track 4.18 -> 55.4 mm, vias 0 -> 3
- net N$100: track 0.00 -> 50.7 mm, vias 0 -> 3
- net N$98: track 0.00 -> 49.1 mm, vias 0 -> 1
- net N$101: track 0.00 -> 49.1 mm, vias 0 -> 2
- net N$108: track 0.00 -> 47.2 mm, vias 0 -> 2
- net PORT18': track 9.22 -> 55.5 mm, vias 0 -> 3
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
Commit message: Added a system description document
Routing:
- net JTAG_TDI: track 0.00 -> 46.3 mm, vias 0 -> 1
- net TXD0: track 0.00 -> 28.4 mm, vias 0 -> 2
- net CC_NHIB: track 45.6 -> 46.6 mm
- net CC_CS: track 55.4 -> 56.4 mm
Changed lines of the file:
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@@
 <grid distance="0.01" unitdist="inch" unit="inch" style="lines" multiple="1" display="no" altdistance="0.0025" altunitdist="inch" altunit="inch"/>
 <layers>
-<layer number="1" name="Top" color="4" fill="1" visible="no" active="yes"/>
+<layer number="1" name="Top" color="4" fill="1" visible="yes" active="yes"/>
 <layer number="2" name="Route2" color="11" fill="1" visible="no" active="yes"/>
 <layer number="3" name="Route3" color="4" fill="3" visible="no" active="no"/>
@@
 <layer number="13" name="Route13" color="4" fill="5" visible="no" active="no"/>
 <layer number="14" name="Route14" color="1" fill="6" visible="no" active="no"/>
-<layer number="15" name="Route15" color="13" fill="1" visible="yes" active="yes"/>
-<layer number="16" name="Bottom" color="1" fill="1" visible="no" active="yes"/>
+<layer number="15" name="Route15" color="13" fill="1" visible="no" active="yes"/>
+<layer number="16" name="Bottom" color="1" fill="1" visible="yes" active="yes"/>
 <layer number="17" name="Pads" color="2" fill="1" visible="yes" active="yes"/>
 <layer number="18" name="Vias" color="2" fill="1" visible="yes" active="yes"/>
 <layer number="19" name="Unrouted" color="6" fill="1" visible="yes" active="yes"/>
 <layer number="20" name="Dimension" color="15" fill="1" visible="yes" active="yes"/>
-<layer number="21" name="tPlace" color="7" fill="1" visible="no" active="yes"/>
-<layer number="22" name="bPlace" color="7" fill="1" visible="no" active="yes"/>
+<layer number="21" name="tPlace" color="7" fill="1" visible="yes" active="yes"/>
+<layer number="22" name="bPlace" color="7" fill="1" visible="yes" active="yes"/>
 <layer number="23" name="tOrigins" color="15" fill="1" visible="no" active="yes"/>
 <layer number="24" name="bOrigins" color="15" fill="1" visible="no" active="yes"/>
-<layer number="25" name="tNames" color="7" fill="1" visible="no" active="yes"/>
-<layer number="26" name="bNames" color="7" fill="1" visible="no" active="yes"/>
+<layer number="25" name="tNames" color="7" fill="1" visible="yes" active="yes"/>
+<layer number="26" name="bNames" color="7" fill="1" visible="yes" active="yes"/>
 <layer number="27" name="tValues" color="7" fill="1" visible="no" active="yes"/>
 <layer number="28" name="bValues" color="7" fill="1" visible="no" active="yes"/>
-<layer number="29" name="tStop" color="7" fill="3" visible="no" active="yes"/>
-<layer number="30" name="bStop" color="7" fill="6" visible="no" active="yes"/>
+<layer number="29" name="tStop" color="7" fill="3" visible="yes" active="yes"/>
+<layer number="30" name="bStop" color="7" fill="6" visible="yes" active="yes"/>
 <layer number="31" name="tCream" color="7" fill="4" visible="no" active="yes"/>
 <layer number="32" name="bCream" color="7" fill="5" visible="no" active="yes"/>
@@
 <layer number="49" name="Reference" color="7" fill="1" visible="no" active="yes"/>
 <layer number="50" name="dxf" color="7" fill="1" visible="no" active="no"/>
-<layer number="51" name="tDocu" color="7" fill="1" visible="no" active="yes"/>
-<layer number="52" name="bDocu" color="7" fill="1" visible="no" active="yes"/>
+<layer number="51" name="tDocu" color="7" fill="1" visible="yes" active="yes"/>
+<layer number="52" name="bDocu" color="7" fill="1" visible="yes" active="yes"/>
 <layer number="53" name="tGND_GNDA" color="7" fill="9" visible="no" active="no"/>
 <layer number="54" name="bGND_GNDA" color="1" fill="9" visible="no" active="no"/>
@@
 <param name="mlMinCreamFrame" value="0mil"/>
 <param name="mlMaxCreamFrame" value="0mil"/>
-<param name="mlViaStopLimit" value="0mil"/>
+<param name="mlViaStopLimit" value="20mil"/>
 <param name="srRoundness" value="0"/>
 <param name="srMinRoundness" value="0mil"/>
@@
 <contactref element="U2" pad="27"/>
 <wire x1="54.25" y1="42.954" x2="54.836" y2="42.954" width="0.1524" layer="1"/>
-<wire x1="54.836" y1="42.954" x2="55.245" y2="42.545" width="0.1524" layer="1"/>
-<wire x1="55.245" y1="42.545" x2="55.245" y2="42.291" width="0.1524" layer="1"/>
-<wire x1="55.245" y1="42.291" x2="55.88" y2="41.656" width="0.1524" layer="1"/>
+<wire x1="54.836" y1="42.954" x2="55.3085" y2="42.4815" width="0.1524" layer="1"/>
+<wire x1="55.3085" y1="42.4815" x2="55.3085" y2="42.2275" width="0.1524" layer="1"/>
+<wire x1="55.3085" y1="42.2275" x2="55.88" y2="41.656" width="0.1524" layer="1"/>
 <via x="55.88" y="41.656" extent="1-16" drill="0.3302"/>
 <wire x1="55.88" y1="41.656" x2="54.1655" y2="43.3705" width="0.1524" layer="15"/>
@@
 <contactref element="R7" pad="7"/>
 <contactref element="U2" pad="26"/>
-<wire x1="54.25" y1="42.454" x2="47.682" y2="60.922" width="0" layer="19" extent="1-1"/>
+<wire x1="54.25" y1="42.454" x2="54.6375" y2="42.454" width="0.1524" layer="1"/>
+<wire x1="54.6375" y1="42.454" x2="55.118" y2="41.9735" width="0.1524" layer="1"/>
+<wire x1="55.118" y1="41.9735" x2="55.118" y2="40.132" width="0.1524" layer="1"/>
+<via x="55.118" y="40.132" extent="1-16" drill="0.3302"/>
+<wire x1="55.118" y1="40.132" x2="54.102" y2="40.132" width="0.1524" layer="16"/>
+<wire x1="54.102" y1="40.132" x2="53.086" y2="41.148" width="0.1524" layer="16"/>
+<wire x1="53.086" y1="41.148" x2="53.086" y2="49.784" width="0.1524" layer="16"/>
+<wire x1="53.086" y1="49.784" x2="53.594" y2="50.292" width="0.1524" layer="16"/>
+<wire x1="53.594" y1="50.292" x2="53.594" y2="50.8" width="0.1524" layer="16"/>
+<wire x1="53.594" y1="50.8" x2="53.34" y2="51.054" width="0.1524" layer="16"/>
+<wire x1="53.34" y1="51.054" x2="52.324" y2="51.054" width="0.1524" layer="16"/>
+<wire x1="52.324" y1="51.054" x2="51.816" y2="51.562" width="0.1524" layer="16"/>
+<wire x1="51.816" y1="51.562" x2="51.816" y2="53.086" width="0.1524" layer="16"/>
+<wire x1="51.816" y1="53.086" x2="48.387" y2="56.515" width="0.1524" layer="16"/>
+<wire x1="48.387" y1="56.515" x2="48.387" y2="57.277" width="0.1524" layer="16"/>
+<via x="48.387" y="57.277" extent="1-16" drill="0.3302"/>
+<wire x1="48.387" y1="57.277" x2="48.387" y2="59.309" width="0.1524" layer="1"/>
+<wire x1="48.387" y1="59.309" x2="48.26" y2="59.436" width="0.1524" layer="1"/>
+<wire x1="48.26" y1="59.436" x2="48.006" y2="59.69" width="0.1524" layer="1"/>
+<wire x1="47.682" y1="60.922" x2="47.682" y2="60.014" width="0.1524" layer="1"/>
+<wire x1="47.682" y1="60.014" x2="48.006" y2="59.69" width="0.1524" layer="1"/>
 </signal>
 <signal name="SCL">
@@
 <contactref element="JP1" pad="8"/>
 <contactref element="U2" pad="25"/>
-<wire x1="54.25" y1="41.954" x2="59.436" y2="65.405" width="0" layer="19" extent="1-1"/>
+<wire x1="54.25" y1="41.954" x2="54.25" y2="39.518" width="0.1524" layer="1"/>
+<wire x1="54.25" y1="39.518" x2="54.356" y2="39.37" width="0.1524" layer="1"/>
+<via x="54.356" y="39.37" extent="1-16" drill="0.3302"/>
+<wire x1="54.356" y1="39.37" x2="55.626" y2="39.37" width="0.1524" layer="16"/>
+<wire x1="55.626" y1="39.37" x2="55.88" y2="39.624" width="0.1524" layer="16"/>
+<wire x1="55.88" y1="39.624" x2="55.88" y2="40.64" width="0.1524" layer="16"/>
+<wire x1="55.88" y1="40.64" x2="55.626" y2="40.894" width="0.1524" layer="16"/>
+<wire x1="55.626" y1="40.894" x2="54.61" y2="40.894" width="0.1524" layer="16"/>
+<wire x1="54.61" y1="40.894" x2="54.102" y2="41.402" width="0.1524" layer="16"/>
+<wire x1="54.102" y1="41.402" x2="54.102" y2="49.784" width="0.1524" layer="16"/>
+<wire x1="54.102" y1="49.784" x2="55.372" y2="51.054" width="0.1524" layer="16"/>
+<wire x1="55.372" y1="51.054" x2="64.262" y2="51.054" width="0.1524" layer="16"/>
+<wire x1="64.262" y1="51.054" x2="65.532" y2="52.324" width="0.1524" layer="16"/>
+<wire x1="65.532" y1="52.324" x2="65.532" y2="63.5" width="0.1524" layer="16"/>
+<wire x1="65.532" y1="63.5" x2="64.77" y2="64.262" width="0.1524" layer="16"/>
+<wire x1="64.77" y1="64.262" x2="60.579" y2="64.262" width="0.1524" layer="16"/>
+<wire x1="60.579" y1="64.262" x2="59.436" y2="65.405" width="0.1524" layer="16"/>
 </signal>
 <signal name="JTAG_RESET">
@@
 <wire x1="55.118" y1="48.26" x2="55.118" y2="47.498" width="0.1524" layer="2"/>
 <wire x1="55.118" y1="47.498" x2="54.356" y2="46.736" width="0.1524" layer="2"/>
-<wire x1="54.356" y1="46.736" x2="54.356" y2="31.115" width="0.1524" layer="2"/>
+<wire x1="54.356" y1="46.736" x2="54.356" y2="41.656" width="0.1524" layer="2"/>
+<wire x1="54.356" y1="41.656" x2="53.086" y2="40.386" width="0.1524" layer="2"/>
+<wire x1="53.086" y1="40.386" x2="53.086" y2="36.83" width="0.1524" layer="2"/>
+<wire x1="53.086" y1="36.83" x2="54.356" y2="35.56" width="0.1524" layer="2"/>
+<wire x1="54.356" y1="35.56" x2="54.356" y2="31.115" width="0.1524" layer="2"/>
 <wire x1="54.356" y1="31.115" x2="54.229" y2="30.988" width="0.1524" layer="2"/>
 <via x="54.229" y="30.988" extent="1-16" drill="0.3302"/>
@@
 <wire x1="55.88" y1="49.022" x2="55.88" y2="47.5615" width="0.1524" layer="2"/>
 <wire x1="55.88" y1="47.5615" x2="54.864" y2="46.5455" width="0.1524" layer="2"/>
-<wire x1="54.864" y1="46.5455" x2="54.864" y2="29.21" width="0.1524" layer="2"/>
+<wire x1="54.864" y1="46.5455" x2="54.864" y2="41.402" width="0.1524" layer="2"/>
+<wire x1="54.864" y1="41.402" x2="53.594" y2="40.132" width="0.1524" layer="2"/>
+<wire x1="53.594" y1="40.132" x2="53.594" y2="37.084" width="0.1524" layer="2"/>
+<wire x1="53.594" y1="37.084" x2="54.864" y2="35.814" width="0.1524" layer="2"/>
+<wire x1="54.864" y1="35.814" x2="54.864" y2="29.21" width="0.1524" layer="2"/>
 <via x="54.864" y="29.21" extent="1-16" drill="0.3302"/>
 <wire x1="54.864" y1="29.21" x2="54.61" y2="29.464" width="0.1524" layer="16"/>
