File: MultiSpork/hardware/MultiSpork-board/MultiSpork-v1.brd (EAGLE design)
At the start: 86.4 x 76.2 mm, 216 parts, among them J1 U.FL, Q2 32.768 kHz, Q3 40 MHz, Q4 MMBT3904, Q5 MMBT3904, SW1 JS102011SAQN, U1 USD-SOCKETNEW, U10 M25PX80, U2 SAM3SA-MU, U3 MAX11300GTL, U4 LT3580EMS8E, U5 LT3580EMS8E, U6 LT3580EMS8E, U7 MCP73831, U8 LT3580EMS8E, U9 CC3100

Commit message: .\s5uqt2as.xa0.txt
Parts:
- C35, C36, C81, C82: value (none) -> 33p
- C37, C42, C48, C54: value (none) -> 4u7
- C38, C43, C49, C55: value (none) -> 100n
- C39, C56: value (none) -> 2n2
- C40, C41, C46, C52, C57, C60, C61, C62: value (none) -> 10u
- C44, C50: value (none) -> 1n
- C45, C51, C58: value (none) -> 1u
- C47, C53: value (none) -> 22p
- C59: value (none) -> DNP
- C83, C84: value (none) -> 15p
- D16, D18, D19: value (none) -> 2A/40V
- F2: value 1500 mA -> 1000 mA
- L3: value L-US2323 -> 3u9
- L4, L5, L6, L7: value L-US1008 -> 2u2
- L8: value L-US2323 -> 5u3
- L9: value L-US1008 -> 5u6
- Q1: value (none) -> 20 MHz
- R1, R16, R19, R22: value (none) -> 47K
- R14: value (none) -> 105K
- R15, R18, R21, R24, R36: value (none) -> 10K
- R17: value (none) -> 45K3
- R20: value (none) -> 24K
- R23: value (none) -> 120K
- R40: value (none) -> 1R
